File: 4x_power_opamp.kicad_sch (KiCad schematic)
At the start: 33 parts, among them J1 jmp, J2 jmp

Commit message: Test pcb done, and made
Parts:
- removed C? (x2): 10u, Capacitor_SMD:C_0805_2012Metric_Pad1.18x1.45mm_HandSolder, symbol Device:C_Small
- removed C? (x2): 100n, Capacitor_SMD:C_0603_1608Metric_Pad1.08x0.95mm_HandSolder, symbol Device:C_Small
- removed C?: 1u, Capacitor_SMD:C_0603_1608Metric_Pad1.08x0.95mm_HandSolder, symbol Device:C_Small
- removed J? (x3): Conn_Coaxial, symbol Connector:Conn_Coaxial
- removed Q?: Q_NPN_BCE, symbol Device:Q_NPN_BCE
- removed U? (x5): Opamp_Quad, symbol Device:Opamp_Quad
- added C11, C13, C15: 100n, Capacitor_SMD:C_0603_1608Metric_Pad1.08x0.95mm_HandSolder, symbol Device:C_Small
- added C12: 1u, Capacitor_SMD:C_0603_1608Metric_Pad1.08x0.95mm_HandSolder, symbol Device:C_Small
- added C2: 100u, Capacitor_SMD:CP_Elec_10x10.5, symbol Device:C_Polarized_Small
- added C4: 10u, Capacitor_SMD:C_0805_2012Metric_Pad1.18x1.45mm_HandSolder, symbol Device:C_Small
- added J5: power, TerminalBlock_MetzConnect:TerminalBlock_MetzConnect_Type094_RT03502HBLU_1x02_P5.00mm_Horizontal, symbol Connector:Conn_01x02_Female
- added J6: test_in, Connector_Coaxial:BNC_Amphenol_B6252HB-NPP3G-50_Horizontal, symbol Connector:Conn_Coaxial
- added Q1: mje15031, Package_TO_SOT_THT:TO-220-3_Vertical, symbol Device:Q_PNP_BCE
- added Q2: 2n5039, Package_TO_SOT_THT:TO-3, symbol Device:Q_NPN_BEC
- added U1: LMH6642MF, Package_TO_SOT_SMD:SOT-23-5, symbol Amplifier_Operational:LMH6609MF
- C1: renamed from C?; footprint (none) -> Capacitor_SMD:CP_Elec_10x10.5
- J1, J2: footprint (none) -> Connector_PinHeader_2.54mm:PinHeader_1x03_P2.54mm_Vertical
- J4: renamed from J?; footprint (none) -> TerminalBlock_MetzConnect:TerminalBlock_MetzConnect_Type094_RT03502HBLU_1x02_P5.00mm_Horizontal
- J7: renamed from J?; footprint (none) -> Connector_Coaxial:BNC_Amphenol_B6252HB-NPP3G-50_Horizontal
- NT1, NT2: renamed from NT?; footprint (none) -> NetTie:NetTie-2_SMD_Pad0.5mm
- R1, R2, R3, R4, R5, R6, R7: renamed from R?; footprint (none) -> Resistor_SMD:R_0603_1608Metric_Pad0.98x0.95mm_HandSolder
- gave numbers to parts that had none: 5
Connections:
- net GND: now also C11.2, C12.2, C13.2, C15.2, C2.2, C4.2, J5.1 (Pin_1), J6.2 (Ext), U1.2 (V-)
- net in0: now also J6.1 (In)
- net in0+: now also U1.3 (+)
- net in0-: now also U1.4 (-)
- net opout0: now also Q1.2 (C), Q2.1 (B); no longer R7.2
- net opout_r0: now also U1.1
- net out0+: now also Q2.2 (E)
- net vin: now also C11.1, C12.1, C13.1, C2.1, C4.1, J5.2 (Pin_2), Q1.3 (E), U1.5 (V+); no longer C1.1, C14.1, C3.1, J4.2 (Pin_2)
- new net opout_base_0: Q1.1 (B), R7.2
- new net vpower: C1.1, C14.1, C15.1, C3.1, J4.2 (Pin_2), Q2.3 (C)
Other:
- note added: "max 5V! (output transistors limit)"
- moved on the sheet: C14, C9, J1, J7, NT1, NT2, R5, R6, R7
